Commit message: Fix typo, add material_yaskawa_white for hc20

File: motoman_hc20_support/urdf/hc20_macro.xacro (robot description, xacro)
@@ -1,9 +1,6 @@
 <?xml version="1.0" ?>
 <robot xmlns:xacro="http://ros.org/wiki/xacro">
+  <xacro:include filename="$(find motoman_resources)/urdf/common_materials.xacro"/>
   <xacro:macro name="motoman_hc20" params="prefix">
-    <!-- Properties -->
-    <material name="yaskawa_white">
-      <color rgba="0.99 0.99 0.99 1" />
-    </material>
     <!-- link list -->
     <link name="${prefix}base_link">
@@ -12,5 +9,5 @@
           <mesh filename="package://motoman_hc20_support/meshes/hc20/visual/base_link.stl"/>
         </geometry>
-        <material name="yaskawa_white"/>
+        <xacro:material_yaskawa_white />
       </visual>
       <collision>
@@ -25,5 +22,5 @@
           <mesh filename="package://motoman_hc20_support/meshes/hc20/visual/link_1_s.stl"/>
         </geometry>
-        <material name="yaskawa_white"/>
+        <xacro:material_yaskawa_white />
       </visual>
       <collision>
@@ -38,5 +35,5 @@
           <mesh filename="package://motoman_hc20_support/meshes/hc20/visual/link_2_l.stl"/>
         </geometry>
-        <material name="yaskawa_white"/>
+        <xacro:material_yaskawa_white />
       </visual>
       <collision>
@@ -51,5 +48,5 @@
           <mesh filename="package://motoman_hc20_support/meshes/hc20/visual/link_3_u.stl"/>
         </geometry>
-        <material name="yaskawa_white"/>
+        <xacro:material_yaskawa_white />
       </visual>
       <collision>
@@ -64,5 +61,5 @@
           <mesh filename="package://motoman_hc20_support/meshes/hc20/visual/link_4_r.stl"/>
         </geometry>
-        <material name="yaskawa_white"/>
+        <xacro:material_yaskawa_white />
       </visual>
       <collision>
@@ -77,5 +74,5 @@
           <mesh filename="package://motoman_hc20_support/meshes/hc20/visual/link_5_b.stl"/>
         </geometry>
-        <material name="yaskawa_white"/>
+        <xacro:material_yaskawa_white />
       </visual>
       <collision>
@@ -90,5 +87,5 @@
           <mesh filename="package://motoman_hc20_support/meshes/hc20/visual/link_6_t.stl"/>
         </geometry>
-        <material name="yaskawa_white"/>
+        <xacro:material_yaskawa_white />
       </visual>
       <collision>

Commit message: added transmissions to the hc20 xacro

File: motoman_hc20_support/urdf/hc20_macro.xacro (robot description, xacro)
@@ -16,4 +16,8 @@
         </geometry>
       </collision>
+      <inertial>
+        <mass value="0.01" />
+        <inertia ixx="0.03" iyy="0.03" izz="0.03" ixy="0.0" ixz="0.0" iyz="0.0" />
+      </inertial>
     </link>
     <link name="${prefix}link_1_s">
@@ -29,4 +33,8 @@
         </geometry>
       </collision>
+      <inertial>
+        <mass value="0.01" />
+        <inertia ixx="0.03" iyy="0.03" izz="0.03" ixy="0.0" ixz="0.0" iyz="0.0" />
+      </inertial>
     </link>
     <link name="${prefix}link_2_l">
@@ -42,4 +50,8 @@
         </geometry>
       </collision>
+      <inertial>
+        <mass value="0.01" />
+        <inertia ixx="0.03" iyy="0.03" izz="0.03" ixy="0.0" ixz="0.0" iyz="0.0" />
+      </inertial>
     </link>
     <link name="${prefix}link_3_u">
@@ -55,4 +67,8 @@
         </geometry>
       </collision>
+      <inertial>
+        <mass value="0.01" />
+        <inertia ixx="0.03" iyy="0.03" izz="0.03" ixy="0.0" ixz="0.0" iyz="0.0" />
+      </inertial>
     </link>
     <link name="${prefix}link_4_r">
@@ -68,4 +84,8 @@
         </geometry>
       </collision>
+      <inertial>
+        <mass value="0.01" />
+        <inertia ixx="0.03" iyy="0.03" izz="0.03" ixy="0.0" ixz="0.0" iyz="0.0" />
+      </inertial>
     </link>
     <link name="${prefix}link_5_b">
@@ -81,4 +101,8 @@
         </geometry>
       </collision>
+      <inertial>
+        <mass value="0.01" />
+        <inertia ixx="0.03" iyy="0.03" izz="0.03" ixy="0.0" ixz="0.0" iyz="0.0" />
+      </inertial>
     </link>
     <link name="${prefix}link_6_t">
@@ -94,4 +118,8 @@
         </geometry>
       </collision>
+      <inertial>
+        <mass value="0.01" />
+        <inertia ixx="0.03" iyy="0.03" izz="0.03" ixy="0.0" ixz="0.0" iyz="0.0" />
+      </inertial>
     </link>
     <link name="${prefix}tool0"/>
@@ -105,4 +133,13 @@
       <limit lower="${radians(-180)}" upper="${radians(180)}" effort="917.28" velocity="${radians(80)}"/>
     </joint>
+    <transmission name="${prefix}joint_1_s_trans">
+          <type>transmission_interface/SimpleTransmission</type>
+          <joint name="${prefix}joint_1_s">
+            <hardwareInterface>hardware_interface/EffortJointInterface</hardwareInterface>
+          </joint>
+          <actuator name="${prefix}joint_1_s_motor">
+            <mechanicalReduction>1</mechanicalReduction>
+          </actuator>
+    </transmission>
     <joint name="${prefix}joint_2_l" type="revolute">
       <parent link="${prefix}link_1_s"/>
@@ -112,4 +149,14 @@
       <limit lower="${radians(-180)}" upper="${radians(180)}" effort="1223.04" velocity="${radians(80)}"/>
     </joint>
+    <transmission name="${prefix}joint_2_l_trans">
+      <type>transmission_interface/SimpleTransmission</type>
+      <joint name="${prefix}joint_2_l">
+        <hardwareInterface>hardware_interface/EffortJointInterface</hardwareInterface>
+      </joint>
+      <actuator name="${prefix}joint_2_l_motor">
+        <hardwareInterface>hardware_interface/EffortJointInterface</hardwareInterface>
+        <mechanicalReduction>1</mechanicalReduction>
+      </actuator>
+    </transmission>
     <joint name="${prefix}joint_3_u" type="revolute">
       <parent link="${prefix}link_2_l"/>
@@ -119,4 +166,14 @@
       <limit lower="${radians(-67)}" upper="${radians(247)}" effort="642.88" velocity="${radians(120)}"/>
     </joint>
+    <transmission name="${prefix}joint_3_u_trans">
+      <type>transmission_interface/SimpleTransmission</type>
+      <joint name="${prefix}joint_3_u">
+        <hardwareInterface>hardware_interface/EffortJointInterface</hardwareInterface>
+      </joint>
+      <actuator name="${prefix}joint_3_u_motor">
+        <hardwareInterface>hardware_interface/EffortJointInterface</hardwareInterface>
+        <mechanicalReduction>1</mechanicalReduction>
+      </actuator>
+    </transmission>
     <joint name="${prefix}joint_4_r" type="revolute">
       <parent link="${prefix}link_3_u"/>
@@ -126,4 +183,14 @@
       <limit lower="${radians(-210)}" upper="${radians(210)}" effort="368.48" velocity="${radians(130)}"/>
     </joint>
+    <transmission name="${prefix}joint_4_r_trans">
+      <type>transmission_interface/SimpleTransmission</type>
+      <joint name="${prefix}joint_4_r">
+        <hardwareInterface>hardware_interface/EffortJointInterface</hardwareInterface>
+      </joint>
+      <actuator name="${prefix}joint_4_r_motor">
+        <hardwareInterface>hardware_interface/EffortJointInterface</hardwareInterface>
+        <mechanicalReduction>1</mechanicalReduction>
+      </actuator>
+    </transmission>
     <joint name="${prefix}joint_5_b" type="revolute">
       <parent link="${prefix}link_4_r"/>
@@ -133,4 +200,14 @@
       <limit lower="${radians(-180)}" upper="${radians(180)}" effort="141.12" velocity="${radians(180)}"/>
     </joint>
+    <transmission name="${prefix}joint_5_b_trans">
+      <type>transmission_interface/SimpleTransmission</type>
+      <joint name="${prefix}joint_5_b">
+        <hardwareInterface>hardware_interface/EffortJointInterface</hardwareInterface>
+      </joint>
+      <actuator name="${prefix}joint_5_b_motor">
+        <hardwareInterface>hardware_interface/EffortJointInterface</hardwareInterface>
+        <mechanicalReduction>1</mechanicalReduction>
+      </actuator>
+    </transmission>
     <joint name="${prefix}joint_6_t" type="revolute">
       <parent link="${prefix}link_5_b"/>
@@ -140,4 +217,14 @@
       <limit lower="${radians(-210)}" upper="${radians(210)}" effort="141.12" velocity="${radians(180)}"/>
     </joint>
+    <transmission name="${prefix}joint_6_t_trans">
+      <type>transmission_interface/SimpleTransmission</type>
+      <joint name="${prefix}joint_6_t">
+        <hardwareInterface>hardware_interface/EffortJointInterface</hardwareInterface>
+      </joint>
+      <actuator name="${prefix}joint_6_t_motor">
+        <hardwareInterface>hardware_interface/EffortJointInterface</hardwareInterface>
+        <mechanicalReduction>1</mechanicalReduction>
+      </actuator>
+    </transmission>
     <joint name="${prefix}joint_6_t-tool0" type="fixed">
       <origin xyz="0.200 0 0" rpy="${radians(180)} ${radians(-90)} 0"/>
